File: MainController/maincontroller/maincontroller.sch (KiCad schematic (older format))
At the start: 30 parts, among them J1 LED, J2 Receiver, J3 5VIN, J4 Analog_Motor, J5 OneWire, J6 Conn_01x04, SW1 SW_Push

Commit message: main controller pcb
Parts:
- added J7: Conn_01x02, Connector_JST:JST_EH_B02B-EH-A_1x02_P2.50mm_Vertical, symbol Connector_Generic:Conn_01x02
- added J8: Conn_01x05_Female, Connector_JST:JST_EH_B05B-EH-A_1x05_P2.50mm_Vertical, symbol Connector:Conn_01x05_Female
- J6: value Conn_01x04 -> Hall_In
- R11, R14: footprint Resistor_THT:R_Axial_DIN0309_L9.0mm_D3.2mm_P12.70mm_Horizontal -> Resistor_THT:R_Axial_DIN0207_L6.3mm_D2.5mm_P2.54mm_Vertical
- R12, R13: footprint Resistor_THT:R_Axial_DIN0309_L9.0mm_D3.2mm_P12.70mm_Horizontal -> Resistor_THT:R_Axial_DIN0309_L9.0mm_D3.2mm_P2.54mm_Vertical
- R15: footprint Resistor_THT:R_Axial_DIN0204_L3.6mm_D1.6mm_P2.54mm_Vertical -> Resistor_THT:R_Axial_DIN0207_L6.3mm_D2.5mm_P7.62mm_Horizontal
- R16, R17, R18: footprint Resistor_THT:R_Axial_DIN0204_L3.6mm_D1.6mm_P2.54mm_Vertical -> Resistor_THT:R_Axial_DIN0309_L9.0mm_D3.2mm_P12.70mm_Horizontal
- R5: footprint Resistor_THT:R_Axial_DIN0204_L3.6mm_D1.6mm_P2.54mm_Vertical -> Resistor_THT:R_Axial_DIN0411_L9.9mm_D3.6mm_P12.70mm_Horizontal
- SW1: footprint Button_Switch_SMD:SW_SPST_B3S-1000 -> Button_Switch_THT:SW_DIP_SPSTx01_Piano_10.8x4.1mm_W7.62mm_P2.54mm
Connections:
- wire segments 177 -> 212
Changed lines of the file:
@@
 EESchema Schematic File Version 4
+LIBS:maincontroller-cache
 EELAYER 26 0
 EELAYER END
@@
 F 0 "SW1" H 5600 5385 50  0000 C CNN
 F 1 "SW_Push" H 5600 5294 50  0000 C CNN
-F 2 "Button_Switch_SMD:SW_SPST_B3S-1000" H 5600 5300 50  0001 C CNN
+F 2 "Button_Switch_THT:SW_DIP_SPSTx01_Piano_10.8x4.1mm_W7.62mm_P2.54mm" H 5600 5300 50  0001 C CNN
 F 3 "" H 5600 5300 50  0001 C CNN
 	1    5600 5100
@@
 	4750 2700 3100 2700
 Wire Wire Line
-	9000 6200 8800 6200
-Wire Wire Line
 	8300 6200 8300 6350
 Wire Wire Line
 	8300 6350 5400 6350
-Wire Wire Line
-	9000 6300 8900 6300
 Wire Wire Line
 	8350 6300 8350 6400
@@
 F 0 "R5" V 3043 6250 50  0000 C CNN
 F 1 "R215" V 3134 6250 50  0000 C CNN
-F 2 "Resistor_THT:R_Axial_DIN0204_L3.6mm_D1.6mm_P2.54mm_Vertical" V 3180 6250 50  0001 C CNN
+F 2 "Resistor_THT:R_Axial_DIN0411_L9.9mm_D3.6mm_P12.70mm_Horizontal" V 3180 6250 50  0001 C CNN
 F 3 "~" H 3250 6250 50  0001 C CNN
 	1    3250 6250
@@
 	1    0    0    -1
 $EndComp
-Wire Wire Line
-	3200 6750 3100 6750
 Connection ~ 3200 6150
 Wire Wire Line
-	3200 6150 3200 6750
-Wire Wire Line
-	3300 5800 3300 6850
-Wire Wire Line
-	3300 6850 3100 6850
+	3300 5800 3300 6750
 Connection ~ 3300 5800
 Wire Wire Line
 	8350 6300 8800 6300
 Wire Wire Line
-	8800 6300 8800 6200
-Connection ~ 8800 6200
-Wire Wire Line
 	8300 6200 8700 6200
 Wire Wire Line
@@
 	8700 6350 8900 6350
 Wire Wire Line
-	8900 6350 8900 6300
-Connection ~ 8900 6300
-Wire Wire Line
 	8900 5600 9200 5600
 Wire Wire Line
-	8900 5600 8900 6300
-Wire Wire Line
 	9250 5650 8800 5650
 Wire Wire Line
-	8800 5650 8800 6200
-Wire Wire Line
-	9000 6000 8500 6000
-Wire Wire Line
-	8500 6100 9000 6100
-Wire Wire Line
-	9000 5900 8500 5900
-Wire Wire Line
-	8500 5800 9000 5800
-Wire Wire Line
 	5400 5200 5400 5400
 Wire Wire Line
-	5900 5400 5400 5400
+	5900 5400 5800 5400
 Wire Wire Line
 	5400 5400 5400 6350
@@
 	8500 2600 9400 2600
 Wire Wire Line
-	9200 2800 9200 5600
+	9200 2800 9200 3600
 Wire Wire Line
 	9200 2800 9400 2800
@@
 P 3950 4100
 F 0 "J6" H 3870 3675 50  0000 C CNN
-F 1 "Conn_01x04" H 3870 3766 50  0000 C CNN
+F 1 "Hall_In" H 3870 3766 50  0000 C CNN
 F 2 "Connector_JST:JST_EH_B04B-EH-A_1x04_P2.50mm_Vertical" H 3950 4100 50  0001 C CNN
 F 3 "~" H 3950 4100 50  0001 C CNN
@@
 F 0 "R11" H 4480 4504 50  0000 R CNN
 F 1 "R2k7" H 4480 4595 50  0000 R CNN
-F 2 "Resistor_THT:R_Axial_DIN0309_L9.0mm_D3.2mm_P12.70mm_Horizontal" V 4480 4550 50  0001 C CNN
+F 2 "Resistor_THT:R_Axial_DIN0207_L6.3mm_D2.5mm_P2.54mm_Vertical" V 4480 4550 50  0001 C CNN
 F 3 "~" H 4550 4550 50  0001 C CNN
 	1    4550 4550
@@
 F 0 "R15" V 5343 3900 50  0000 C CNN
 F 1 "R4k7" V 5434 3900 50  0000 C CNN
-F 2 "Resistor_THT:R_Axial_DIN0204_L3.6mm_D1.6mm_P2.54mm_Vertical" V 5480 3900 50  0001 C CNN
+F 2 "Resistor_THT:R_Axial_DIN0207_L6.3mm_D2.5mm_P7.62mm_Horizontal" V 5480 3900 50  0001 C CNN
 F 3 "~" H 5550 3900 50  0001 C CNN
 	1    5550 3900
@@
 F 0 "R16" V 5343 4000 50  0000 C CNN
 F 1 "R4k7" V 5434 4000 50  0000 C CNN
-F 2 "Resistor_THT:R_Axial_DIN0204_L3.6mm_D1.6mm_P2.54mm_Vertical" V 5480 4000 50  0001 C CNN
+F 2 "Resistor_THT:R_Axial_DIN0309_L9.0mm_D3.2mm_P12.70mm_Horizontal" V 5480 4000 50  0001 C CNN
 F 3 "~" H 5550 4000 50  0001 C CNN
 	1    5550 4000
@@
 F 0 "R17" V 5343 4100 50  0000 C CNN
 F 1 "R4k7" V 5434 4100 50  0000 C CNN
-F 2 "Resistor_THT:R_Axial_DIN0204_L3.6mm_D1.6mm_P2.54mm_Vertical" V 5480 4100 50  0001 C CNN
+F 2 "Resistor_THT:R_Axial_DIN0309_L9.0mm_D3.2mm_P12.70mm_Horizontal" V 5480 4100 50  0001 C CNN
 F 3 "~" H 5550 4100 50  0001 C CNN
 	1    5550 4100
@@
 F 0 "R18" V 5343 4200 50  0000 C CNN
 F 1 "R4k7" V 5434 4200 50  0000 C CNN
-F 2 "Resistor_THT:R_Axial_DIN0204_L3.6mm_D1.6mm_P2.54mm_Vertical" V 5480 4200 50  0001 C CNN
+F 2 "Resistor_THT:R_Axial_DIN0309_L9.0mm_D3.2mm_P12.70mm_Horizontal" V 5480 4200 50  0001 C CNN
 F 3 "~" H 5550 4200 50  0001 C CNN
 	1    5550 4200
 	0    1    1    0
 $EndComp
-Wire Wire Line
-	5900 3700 5700 3700
-Wire Wire Line
-	5700 3700 5700 3900
-Wire Wire Line
-	5900 3800 5750 3800
-Wire Wire Line
-	5750 3800 5750 4000
-Wire Wire Line
-	5750 4000 5700 4000
-Wire Wire Line
-	5900 3900 5800 3900
-Wire Wire Line
-	5800 3900 5800 4100
-Wire Wire Line
-	5800 4100 5700 4100
-Wire Wire Line
-	5900 4000 5850 4000
-Wire Wire Line
-	5850 4000 5850 4200
-Wire Wire Line
-	5850 4200 5700 4200
 $Comp
 L Device:R R8
@@
 F 0 "R12" H 4580 4504 50  0000 R CNN
 F 1 "R2k7" H 4580 4595 50  0000 R CNN
-F 2 "Resistor_THT:R_Axial_DIN0309_L9.0mm_D3.2mm_P12.70mm_Horizontal" V 4580 4550 50  0001 C CNN
+F 2 "Resistor_THT:R_Axial_DIN0309_L9.0mm_D3.2mm_P2.54mm_Vertical" V 4580 4550 50  0001 C CNN
 F 3 "~" H 4650 4550 50  0001 C CNN
 	1    4650 4550
@@
 F 0 "R13" H 4680 4504 50  0000 R CNN
 F 1 "R2k7" H 4680 4595 50  0000 R CNN
-F 2 "Resistor_THT:R_Axial_DIN0309_L9.0mm_D3.2mm_P12.70mm_Horizontal" V 4680 4550 50  0001 C CNN
+F 2 "Resistor_THT:R_Axial_DIN0309_L9.0mm_D3.2mm_P2.54mm_Vertical" V 4680 4550 50  0001 C CNN
 F 3 "~" H 4750 4550 50  0001 C CNN
 	1    4750 4550
@@
 F 0 "R14" H 4780 4504 50  0000 R CNN
 F 1 "R2k7" H 4780 4595 50  0000 R CNN
-F 2 "Resistor_THT:R_Axial_DIN0309_L9.0mm_D3.2mm_P12.70mm_Horizontal" V 4780 4550 50  0001 C CNN
+F 2 "Resistor_THT:R_Axial_DIN0207_L6.3mm_D2.5mm_P2.54mm_Vertical" V 4780 4550 50  0001 C CNN
 F 3 "~" H 4850 4550 50  0001 C CNN
 	1    4850 4550
@@
 Wire Wire Line
 	4550 3900 5400 3900
+Wire Wire Line
+	3200 6850 3100 6850
+Wire Wire Line
+	3200 6750 3200 6850
+Wire Wire Line
+	3200 6700 3200 6750
+Wire Wire Line
+	3100 6750 3300 6750
+Wire Wire Line
+	3200 6150 3200 6750
+Wire Wire Line
+	5700 4200 5750 4200
+Wire Wire Line
+	5700 4100 5800 4100
+Wire Wire Line
+	5950 4000 5900 4000
+Wire Wire Line
+	5850 3900 5900 3900
+Wire Wire Line
+	5850 4000 5850 3900
+Wire Wire Line
+	5700 4000 5850 4000
+Wire Wire Line
+	5700 3900 5700 3750
+Wire Wire Line
+	5700 3750 5950 3750
+Wire Wire Line
+	5950 3750 5950 4000
+Wire Wire Line
+	5750 3800 5750 4200
+Wire Wire Line
+	5750 3800 5900 3800
+Wire Wire Line
+	5800 4100 5800 3700
+Wire Wire Line
+	5800 3700 5900 3700
+Wire Wire Line
+	8750 5800 8500 5800
+$Comp
+L Connector_Generic:Conn_01x02 J7
+U 1 1 5BC4BCB9
+P 5450 2850
+F 0 "J7" H 5370 2525 50  0000 C CNN
+F 1 "Conn_01x02" H 5370 2616 50  0000 C CNN
+F 2 "Connector_JST:JST_EH_B02B-EH-A_1x02_P2.50mm_Vertical" H 5450 2850 50  0001 C CNN
+F 3 "~" H 5450 2850 50  0001 C CNN
+	1    5450 2850
+	-1   0    0    1
+$EndComp
+Wire Wire Line
+	5900 2800 5800 2800
+Wire Wire Line
+	5800 2800 5800 2750
+Wire Wire Line
+	5800 2750 5650 2750
+Wire Wire Line
+	5650 2850 5900 2850
+Wire Wire Line
+	5900 2850 5900 2900
+$Comp
+L Connector:Conn_01x05_Female J8
+U 1 1 5BBFA89A
+P 9700 3400
+F 0 "J8" H 9727 3426 50  0000 L CNN
+F 1 "Conn_01x05_Female" H 9727 3335 50  0000 L CNN
+F 2 "Connector_JST:JST_EH_B05B-EH-A_1x05_P2.50mm_Vertical" H 9700 3400 50  0001 C CNN
+F 3 "~" H 9700 3400 50  0001 C CNN
+	1    9700 3400
+	1    0    0    -1
+$EndComp
+Wire Wire Line
+	9500 3200 9500 3300
+Wire Wire Line
+	9500 3200 9100 3200
+Wire Wire Line
+	9100 3200 9100 2800
+Wire Wire Line
+	9100 2800 8500 2800
+Connection ~ 9500 3200
+Wire Wire Line
+	8500 2900 9000 2900
+Wire Wire Line
+	9000 3400 9500 3400
+Wire Wire Line
+	9000 2900 9000 3400
+Wire Wire Line
+	9500 3500 9500 3400
+Connection ~ 9500 3400
+Wire Wire Line
+	9500 3600 9200 3600
+Connection ~ 9200 3600
+Wire Wire Line
+	9200 3600 9200 5600
+Wire Wire Line
+	9000 5800 8950 5800
+Wire Wire Line
+	8950 5800 8950 5850
+Wire Wire Line
+	8950 5850 8550 5850
+Wire Wire Line
+	8550 5850 8550 6000
+Wire Wire Line
+	8550 6000 8500 6000
+Wire Wire Line
+	9000 5900 8750 5900
+Wire Wire Line
+	8750 5900 8750 5800
+Wire Wire Line
+	9000 6000 8700 6000
+Wire Wire Line
+	8700 6000 8700 5900
+Wire Wire Line
+	8700 5900 8500 5900
+Wire Wire Line
+	9000 6100 8500 6100
+Wire Wire Line
+	5900 5300 5800 5300
+Wire Wire Line
+	5800 5300 5800 5400
+Connection ~ 5800 5400
+Wire Wire Line
+	5800 5400 5400 5400
+Wire Wire Line
+	5900 5200 5800 5200
+Wire Wire Line
+	5800 5200 5800 5300
+Connection ~ 5800 5300
+Wire Wire Line
+	5900 5500 5800 5500
+Wire Wire Line
+	5800 5500 5800 5400
+Wire Wire Line
+	5900 5600 5800 5600
+Wire Wire Line
+	5800 5600 5800 5500
+Connection ~ 5800 5500
+Wire Wire Line
+	8800 5650 8800 6300
+Wire Wire Line
+	8900 5600 8900 6200
+Wire Wire Line
+	9000 6300 8800 6300
+Connection ~ 8800 6300
+Wire Wire Line
+	9000 6200 8900 6200
+Connection ~ 8900 6200
+Wire Wire Line
+	8900 6200 8900 6350
 $EndSCHEMATC

Commit message: removed 5v in, use reciver power instead, simplified relay connector, added reverse pin to motorconnector
Parts:
- removed J3: 5VIN, Connector_JST:JST_EH_B03B-EH-A_1x03_P2.50mm_Vertical, symbol Connector:Conn_01x03_Male
- J4: footprint Connector_PinHeader_2.54mm:PinHeader_1x04_P2.54mm_Vertical -> Connector_PinHeader_2.54mm:PinHeader_1x05_P2.54mm_Vertical; symbol Connector:Conn_01x04_Female -> Connector:Conn_01x05_Female
- J6: footprint Connector_JST:JST_EH_B04B-EH-A_1x04_P2.50mm_Vertical -> Connector_JST:JST_EH_B04B-EH-A_1x05_P2.50mm_Vertical
- relays1: renamed from J8; footprint Connector_JST:JST_EH_B05B-EH-A_1x05_P2.50mm_Vertical -> Connector_PinHeader_2.54mm:PinHeader_1x03_P2.54mm_Vertical; symbol Connector:Conn_01x05_Female -> Connector:Conn_01x03_Female
- renumbered J7 to Bus1, SW1 to Reset1
Connections:
- wire segments 212 -> 210
Changed lines of the file:
@@
 $EndDescr
 $Comp
-L Switch:SW_Push SW1
+L Switch:SW_Push Reset1
 U 1 1 5BB7D413
 P 5600 5100
-F 0 "SW1" H 5600 5385 50  0000 C CNN
+F 0 "Reset1" H 5600 5385 50  0000 C CNN
 F 1 "SW_Push" H 5600 5294 50  0000 C CNN
 F 2 "Button_Switch_THT:SW_DIP_SPSTx01_Piano_10.8x4.1mm_W7.62mm_P2.54mm" H 5600 5300 50  0001 C CNN
@@
 $EndComp
 $Comp
-L Connector:Conn_01x04_Female J4
+L Connector:Conn_01x05_Female J4
 U 1 1 5BB7E5BD
 P 2050 3350
 F 0 "J4" H 2077 3326 50  0000 L CNN
 F 1 "Analog_Motor" H 2077 3235 50  0000 L CNN
-F 2 "Connector_PinHeader_2.54mm:PinHeader_1x04_P2.54mm_Vertical" H 2050 3350 50  0001 C CNN
+F 2 "Connector_PinHeader_2.54mm:PinHeader_1x05_P2.54mm_Vertical" H 2050 3350 50  0001 C CNN
 F 3 "~" H 2050 3350 50  0001 C CNN
 	1    2050 3350
@@
 Wire Wire Line
 	3800 5900 3800 3750
-$Comp
-L Connector:Conn_01x03_Male J3
-U 1 1 5BBE531C
-P 2900 6750
-F 0 "J3" H 3006 7028 50  0000 C CNN
-F 1 "5VIN" H 3006 6937 50  0000 C CNN
-F 2 "Connector_JST:JST_EH_B03B-EH-A_1x03_P2.50mm_Vertical" H 2900 6750 50  0001 C CNN
-F 3 "~" H 2900 6750 50  0001 C CNN
-	1    2900 6750
-	1    0    0    -1
-$EndComp
-Connection ~ 3200 6150
-Wire Wire Line
-	3300 5800 3300 6750
-Connection ~ 3300 5800
 Wire Wire Line
 	8350 6300 8800 6300
@@
 F 0 "J6" H 3870 3675 50  0000 C CNN
 F 1 "Hall_In" H 3870 3766 50  0000 C CNN
-F 2 "Connector_JST:JST_EH_B04B-EH-A_1x04_P2.50mm_Vertical" H 3950 4100 50  0001 C CNN
+F 2 "Connector_JST:JST_EH_B04B-EH-A_1x05_P2.50mm_Vertical" H 3950 4100 50  0001 C CNN
 F 3 "~" H 3950 4100 50  0001 C CNN
 	1    3950 4100
@@
 	4550 3900 5400 3900
 Wire Wire Line
-	3200 6850 3100 6850
-Wire Wire Line
-	3200 6750 3200 6850
-Wire Wire Line
-	3200 6700 3200 6750
-Wire Wire Line
-	3100 6750 3300 6750
-Wire Wire Line
-	3200 6150 3200 6750
-Wire Wire Line
 	5700 4200 5750 4200
 Wire Wire Line
@@
 	8750 5800 8500 5800
 $Comp
-L Connector_Generic:Conn_01x02 J7
+L Connector_Generic:Conn_01x02 Bus1
 U 1 1 5BC4BCB9
 P 5450 2850
-F 0 "J7" H 5370 2525 50  0000 C CNN
+F 0 "Bus1" H 5370 2525 50  0000 C CNN
 F 1 "Conn_01x02" H 5370 2616 50  0000 C CNN
 F 2 "Connector_JST:JST_EH_B02B-EH-A_1x02_P2.50mm_Vertical" H 5450 2850 50  0001 C CNN
@@
 	5900 2850 5900 2900
 $Comp
-L Connector:Conn_01x05_Female J8
+L Connector:Conn_01x03_Female relays1
 U 1 1 5BBFA89A
 P 9700 3400
-F 0 "J8" H 9727 3426 50  0000 L CNN
+F 0 "relays1" H 9727 3426 50  0000 L CNN
 F 1 "Conn_01x05_Female" H 9727 3335 50  0000 L CNN
-F 2 "Connector_JST:JST_EH_B05B-EH-A_1x05_P2.50mm_Vertical" H 9700 3400 50  0001 C CNN
+F 2 "Connector_PinHeader_2.54mm:PinHeader_1x03_P2.54mm_Vertical" H 9700 3400 50  0001 C CNN
 F 3 "~" H 9700 3400 50  0001 C CNN
 	1    9700 3400
@@
 $EndComp
 Wire Wire Line
-	9500 3200 9500 3300
-Wire Wire Line
 	9500 3200 9100 3200
 Wire Wire Line
@@
 Wire Wire Line
 	9100 2800 8500 2800
-Connection ~ 9500 3200
 Wire Wire Line
 	8500 2900 9000 2900
@@
 Wire Wire Line
 	9000 2900 9000 3400
-Wire Wire Line
-	9500 3500 9500 3400
-Connection ~ 9500 3400
 Wire Wire Line
 	9500 3600 9200 3600
@@
 Wire Wire Line
 	8900 6200 8900 6350
+Wire Wire Line
+	5900 4100 5950 4100
+Wire Wire Line
+	5950 4100 5950 4750
+Wire Wire Line
+	5950 4750 2250 4750
+Wire Wire Line
+	2250 4750 2250 3550
+Wire Wire Line
+	9500 3500 9500 3600
+Wire Wire Line
+	9500 3300 9500 3200
 $EndSCHEMATC

Commit message: Meh, doesnt work
Parts:
- Bus1: symbol Connector_Generic:Conn_01x02 -> maincontroller-rescue:Conn_01x02-Connector_Generic
- Hinten_links1, Hinten_rechts1, Vorne_links1, Vorne_rechts1: symbol MCP4725:MCP4725 -> maincontroller-rescue:MCP4725-MCP4725
- J1, J5, J6: symbol Connector_Generic:Conn_01x04 -> maincontroller-rescue:Conn_01x04-Connector_Generic
- J2: symbol Connector_Generic:Conn_01x06 -> maincontroller-rescue:Conn_01x06-Connector_Generic
- J4: symbol Connector:Conn_01x05_Female -> maincontroller-rescue:Conn_01x05_Female-Connector
- R1, R10, R11, R12, R13, R14, R15, R16, R17, R18, R2, R3, R4, R5, R6, R7, R8, R9: symbol Device:R -> maincontroller-rescue:R-Device
- Reset1: symbol Switch:SW_Push -> maincontroller-rescue:SW_Push-Switch
- XA1: symbol arduino:Arduino_Mega2560_Shield -> maincontroller-rescue:Arduino_Mega2560_Shield-arduino
- relays1: value Conn_01x05_Female -> Conn_01x05_Female-Connector; symbol Connector:Conn_01x03_Female -> maincontroller-rescue:Conn_01x05_Female-Connector
Changed lines of the file:
@@
 $EndDescr
 $Comp
-L Switch:SW_Push Reset1
+L maincontroller-rescue:SW_Push-Switch Reset1
 U 1 1 5BB7D413
 P 5600 5100
@@
 $EndComp
 $Comp
-L Connector_Generic:Conn_01x06 J2
+L maincontroller-rescue:Conn_01x06-Connector_Generic J2
 U 1 1 5BB7E71D
 P 9200 6000
@@
 $EndComp
 $Comp
-L arduino:Arduino_Mega2560_Shield XA1
+L maincontroller-rescue:Arduino_Mega2560_Shield-arduino XA1
 U 1 1 5BB7EBA8
 P 7200 3950
@@
 $EndComp
 $Comp
-L Connector_Generic:Conn_01x04 J5
+L maincontroller-rescue:Conn_01x04-Connector_Generic J5
 U 1 1 5BB7F576
 P 2900 6250
@@
 $EndComp
 $Comp
-L Connector:Conn_01x05_Female J4
+L maincontroller-rescue:Conn_01x05_Female-Connector J4
 U 1 1 5BB7E5BD
 P 2050 3350
@@
 $EndComp
 $Comp
-L Connector_Generic:Conn_01x04 J1
+L maincontroller-rescue:Conn_01x04-Connector_Generic J1
 U 1 1 5BB80B10
 P 9600 2600
@@
 $EndComp
 $Comp
-L MCP4725:MCP4725 Vorne_links1
+L maincontroller-rescue:MCP4725-MCP4725 Vorne_links1
 U 1 1 5BB8C41D
 P 2750 2600
@@
 $EndComp
 $Comp
-L MCP4725:MCP4725 Vorne_rechts1
+L maincontroller-rescue:MCP4725-MCP4725 Vorne_rechts1
 U 1 1 5BB8C793
 P 2750 3500
@@
 $EndComp
 $Comp
-L MCP4725:MCP4725 Hinten_links1
+L maincontroller-rescue:MCP4725-MCP4725 Hinten_links1
 U 1 1 5BB8C852
 P 2750 4400
@@
 $EndComp
 $Comp
-L MCP4725:MCP4725 Hinten_rechts1
+L maincontroller-rescue:MCP4725-MCP4725 Hinten_rechts1
 U 1 1 5BB8C992
 P 2750 5300
@@
 Connection ~ 5400 5200
 $Comp
-L Device:R R1
+L maincontroller-rescue:R-Device R1
 U 1 1 5BB91DD8
 P 3250 3000
@@
 $EndComp
 $Comp
-L Device:R R2
+L maincontroller-rescue:R-Device R2
 U 1 1 5BB922C9
 P 3250 3900
@@
 $EndComp
 $Comp
-L Device:R R3
+L maincontroller-rescue:R-Device R3
 U 1 1 5BB9238D
 P 3250 4800
@@
 $EndComp
 $Comp
-L Device:R R4
+L maincontroller-rescue:R-Device R4
 U 1 1 5BB923E1
 P 3250 5700
@@
 	5300 5800 4100 5800
 $Comp
-L Device:R R5
+L maincontroller-rescue:R-Device R5
 U 1 1 5BBD15F0
 P 3250 6250
@@
 	3800 6350 3800 5900
 $Comp
-L Device:R R6
+L maincontroller-rescue:R-Device R6
 U 1 1 5BBDE040
 P 3950 5900
@@
 	5850 2950 5850 3100
 $Comp
-L Connector_Generic:Conn_01x04 J6
+L maincontroller-rescue:Conn_01x04-Connector_Generic J6
 U 1 1 5BD2D1DF
 P 3950 4100
@@
 $EndComp
 $Comp
-L Device:R R11
+L maincontroller-rescue:R-Device R11
 U 1 1 5BD2D2C8
 P 4550 4550
@@
 $EndComp
 $Comp
-L Device:R R7
+L maincontroller-rescue:R-Device R7
 U 1 1 5BD32A4E
 P 4300 3900
@@
 $EndComp
 $Comp
-L Device:R R15
+L maincontroller-rescue:R-Device R15
 U 1 1 5BD32B64
 P 5550 3900
@@
 	5450 3750 5450 3000
 $Comp
-L Device:R R16
+L maincontroller-rescue:R-Device R16
 U 1 1 5BD4DE20
 P 5550 4000
@@
 $EndComp
 $Comp
-L Device:R R17
+L maincontroller-rescue:R-Device R17
 U 1 1 5BD4DE60
 P 5550 4100
@@
 $EndComp
 $Comp
-L Device:R R18
+L maincontroller-rescue:R-Device R18
 U 1 1 5BD4DE9E
 P 5550 4200
@@
 $EndComp
 $Comp
-L Device:R R8
+L maincontroller-rescue:R-Device R8
 U 1 1 5BD88C7C
 P 4300 4000
@@
 $EndComp
 $Comp
-L Device:R R9
+L maincontroller-rescue:R-Device R9
 U 1 1 5BD88CBE
 P 4300 4100
@@
 $EndComp
 $Comp
-L Device:R R10
+L maincontroller-rescue:R-Device R10
 U 1 1 5BD88D02
 P 4300 4200
@@
 $EndComp
 $Comp
-L Device:R R12
+L maincontroller-rescue:R-Device R12
 U 1 1 5BD88DC2
 P 4650 4550
@@
 $EndComp
 $Comp
-L Device:R R13
+L maincontroller-rescue:R-Device R13
 U 1 1 5BD88E0A
 P 4750 4550
@@
 $EndComp
 $Comp
-L Device:R R14
+L maincontroller-rescue:R-Device R14
 U 1 1 5BD88E58
 P 4850 4550
@@
 	8750 5800 8500 5800
 $Comp
-L Connector_Generic:Conn_01x02 Bus1
+L maincontroller-rescue:Conn_01x02-Connector_Generic Bus1
 U 1 1 5BC4BCB9
 P 5450 2850
@@
 	5900 2850 5900 2900
 $Comp
-L Connector:Conn_01x03_Female relays1
+L maincontroller-rescue:Conn_01x05_Female-Connector relays1
 U 1 1 5BBFA89A
 P 9700 3400
 F 0 "relays1" H 9727 3426 50  0000 L CNN
-F 1 "Conn_01x05_Female" H 9727 3335 50  0000 L CNN
+F 1 "Conn_01x05_Female-Connector" H 9727 3335 50  0000 L CNN
 F 2 "Connector_PinHeader_2.54mm:PinHeader_1x03_P2.54mm_Vertical" H 9700 3400 50  0001 C CNN
 F 3 "~" H 9700 3400 50  0001 C CNN
